File: encoder.kicad_pcb (KiCad board)
At the start: 2 copper layers, 40 x 40 mm, 12 parts, among them J1 BM04B-SURS-TFLFSN, U1 AS5600-ASOT

Commit message: added frame
Other:
- board size 40 x 40 mm -> 50 x 50 mm
Changed lines of the file:
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@@
       (effects (font (size 1 1) (thickness 0.15) italic))
     )
-    (fp_line (start 2 1.2) (end 2 -1) (layer "Dwgs.User") (width 0.12))
-    (fp_line (start -2 -1) (end -2 1.2) (layer "Dwgs.User") (width 0.12))
-    (fp_arc (start -2.000001 1.200001) (mid -0.000001 0.998001) (end 1.999999 1.200001) (layer "Dwgs.User") (width 0.12))
     (pad "" np_thru_hole circle (at -1.532737 0.865248) (size 0.6 0.6) (drill 0.5) (layers *.Cu *.Mask))
     (pad "" np_thru_hole circle (at -0.768531 0.778853) (size 0.6 0.6) (drill 0.5) (layers *.Cu *.Mask))
@@
       (effects (font (size 1 1) (thickness 0.15)))
     )
-    (fp_text value "MountingHole" (at 0 3.25) (layer "F.Fab")
+    (fp_text value "MountingHole" (at 0 3.25) (layer "F.Fab") hide
       (effects (font (size 1 1) (thickness 0.15)))
     )
@@
       (effects (font (size 1 1) (thickness 0.15)))
     )
-    (fp_text value "MountingHole" (at 0 3.25) (layer "F.Fab")
+    (fp_text value "MountingHole" (at 0 3.25) (layer "F.Fab") hide
       (effects (font (size 1 1) (thickness 0.15)))
     )
@@
       (effects (font (size 1 1) (thickness 0.15) italic))
     )
-    (fp_line (start 2 1.2) (end 2 -1) (layer "Dwgs.User") (width 0.12))
-    (fp_line (start -2 -1) (end -2 1.2) (layer "Dwgs.User") (width 0.12))
-    (fp_arc (start -2.000001 1.200001) (mid -0.000001 0.998001) (end 1.999999 1.200001) (layer "Dwgs.User") (width 0.12))
     (pad "" np_thru_hole circle (at -1.532737 0.865248 90) (size 0.6 0.6) (drill 0.5) (layers *.Cu *.Mask))
     (pad "" np_thru_hole circle (at -0.768531 0.778853 90) (size 0.6 0.6) (drill 0.5) (layers *.Cu *.Mask))
@@
       (effects (font (size 1 1) (thickness 0.15) italic))
     )
-    (fp_line (start 2 1.2) (end 2 -1) (layer "Dwgs.User") (width 0.12))
-    (fp_line (start -2 -1) (end -2 1.2) (layer "Dwgs.User") (width 0.12))
-    (fp_arc (start -2.000001 1.200001) (mid -0.000001 0.998001) (end 1.999999 1.200001) (layer "Dwgs.User") (width 0.12))
     (pad "" np_thru_hole circle (at -1.532737 0.865248 180) (size 0.6 0.6) (drill 0.5) (layers *.Cu *.Mask))
     (pad "" np_thru_hole circle (at -0.768531 0.778853 180) (size 0.6 0.6) (drill 0.5) (layers *.Cu *.Mask))
@@
       (effects (font (size 1 1) (thickness 0.15) italic))
     )
-    (fp_line (start 2 1.2) (end 2 -1) (layer "Dwgs.User") (width 0.12))
-    (fp_line (start -2 -1) (end -2 1.2) (layer "Dwgs.User") (width 0.12))
-    (fp_arc (start -2.000001 1.200001) (mid -0.000001 0.998001) (end 1.999999 1.200001) (layer "Dwgs.User") (width 0.12))
     (pad "" np_thru_hole circle (at -1.532737 0.865248 270) (size 0.6 0.6) (drill 0.5) (layers *.Cu *.Mask))
     (pad "" np_thru_hole circle (at -0.768531 0.778853 270) (size 0.6 0.6) (drill 0.5) (layers *.Cu *.Mask))
@@
   (gr_line (start 13.55 2) (end 13.55 13.525) (layer "Edge.Cuts") (width 0.1))
   (gr_line (start -2 13.55) (end -13.525 13.55) (layer "Edge.Cuts") (width 0.1))
-  (gr_circle (center 0 0) (end 11.5 0) (layer "Edge.Cuts") (width 0.1) (fill none))
+  (gr_arc (start -11.324999 -2) (mid -8.1319 -8.1319) (end -2 -11.324999) (layer "Edge.Cuts") (width 0.1))
   (gr_line (start 13.55 13.525) (end 2 13.525) (layer "Edge.Cuts") (width 0.1))
-  (gr_rect (start -20 -20) (end 20 20) (layer "Edge.Cuts") (width 0.15) (fill none))
-  (gr_line (start 2 -13.5625) (end 2 -11.3375) (layer "Edge.Cuts") (width 0.1))
+  (gr_rect (start -25 -25) (end 25 25) (layer "Edge.Cuts") (width 0.15) (fill none))
+  (gr_line (start 2 -13.5625) (end 2 -11.324999) (layer "Edge.Cuts") (width 0.1))
   (gr_line (start -2 13.55) (end -2 11.325) (layer "Edge.Cuts") (width 0.1))
   (gr_line (start 2 13.525) (end 2 11.325) (layer "Edge.Cuts") (width 0.1))
-  (gr_line (start -13.525 13.55) (end -13.525 2) (layer "Edge.Cuts") (width 0.1))
+  (gr_line (start -13.525 13.55) (end -13.525 1.995727) (layer "Edge.Cuts") (width 0.1))
   (gr_line (start -2 -13.525) (end -2 -11.325) (layer "Edge.Cuts") (width 0.1))
   (gr_line (start 2 -13.5625) (end 13.525 -13.5625) (layer "Edge.Cuts") (width 0.1))
@@
   (gr_line (start -13.55 -2) (end -11.325 -2) (layer "Edge.Cuts") (width 0.1))
   (gr_line (start 13.525 -2.0125) (end 11.325 -2.0125) (layer "Edge.Cuts") (width 0.1))
+  (gr_arc (start -2 11.324999) (mid -8.133434 8.130366) (end -11.325753 1.995727) (layer "Edge.Cuts") (width 0.1))
+  (gr_arc (start 2 -11.324999) (mid 8.127548 -8.13625) (end 11.322853 -2.012118) (layer "Edge.Cuts") (width 0.1))
   (gr_line (start -13.55 -13.525) (end -2 -13.525) (layer "Edge.Cuts") (width 0.1))
   (gr_line (start 13.525 -13.5625) (end 13.525 -2.0125) (layer "Edge.Cuts") (width 0.1))
-  (gr_line (start -13.525 2) (end -11.35 2) (layer "Edge.Cuts") (width 0.1))
+  (gr_arc (start 11.324999 2) (mid 8.1319 8.1319) (end 2 11.324999) (layer "Edge.Cuts") (width 0.1))
+  (gr_line (start -13.525 1.995727) (end -11.325753 1.995727) (layer "Edge.Cuts") (width 0.1))
   (gr_circle (center 0 0) (end 7 0) (layer "F.Fab") (width 0.1) (fill none))
   (gr_text "Gordon Lay\nLui H-P" (at -4.125 -6 270) (layer "B.SilkS")

Commit message: gigvkhkhnk
Routing:
- added copper zone on F.Cu, net +3.3V
- added copper zone on B.Cu, net GND
- removed copper zone on B.Cu, net +3.3V
- removed copper zone on F.Cu, net GND
Changed lines of the file:
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@@
       (effects (font (size 1 1) (thickness 0.15) italic))
     )
-    (pad "" np_thru_hole circle (at -1.532737 0.865248 90) (size 0.6 0.6) (drill 0.5) (layers *.Cu *.Mask))
     (pad "" np_thru_hole circle (at -0.768531 0.778853 90) (size 0.6 0.6) (drill 0.5) (layers *.Cu *.Mask))
+    (pad "" np_thru_hole circle (at 1.532737 0.865248 90) (size 0.6 0.6) (drill 0.5) (layers *.Cu *.Mask))
     (pad "" np_thru_hole circle (at 0.768531 0.778853 90) (size 0.6 0.6) (drill 0.5) (layers *.Cu *.Mask))
     (pad "" np_thru_hole circle (at 0 0.75 90) (size 0.6 0.6) (drill 0.5) (layers *.Cu *.Mask))
-    (pad "" np_thru_hole circle (at 1.532737 0.865248 90) (size 0.6 0.6) (drill 0.5) (layers *.Cu *.Mask))
+    (pad "" np_thru_hole circle (at -1.532737 0.865248 90) (size 0.6 0.6) (drill 0.5) (layers *.Cu *.Mask))
   )
   (footprint "Capacitor_SMD:C_0603_1608Metric" (layer "F.Cu")
@@
       (effects (font (size 1 1) (thickness 0.15) italic))
     )
+    (pad "" np_thru_hole circle (at -0.768531 0.778853 180) (size 0.6 0.6) (drill 0.5) (layers *.Cu *.Mask))
+    (pad "" np_thru_hole circle (at 1.532737 0.865248 180) (size 0.6 0.6) (drill 0.5) (layers *.Cu *.Mask))
     (pad "" np_thru_hole circle (at -1.532737 0.865248 180) (size 0.6 0.6) (drill 0.5) (layers *.Cu *.Mask))
-    (pad "" np_thru_hole circle (at -0.768531 0.778853 180) (size 0.6 0.6) (drill 0.5) (layers *.Cu *.Mask))
+    (pad "" np_thru_hole circle (at 0 0.75 180) (size 0.6 0.6) (drill 0.5) (layers *.Cu *.Mask))
     (pad "" np_thru_hole circle (at 0.768531 0.778853 180) (size 0.6 0.6) (drill 0.5) (layers *.Cu *.Mask))
-    (pad "" np_thru_hole circle (at 0 0.75 180) (size 0.6 0.6) (drill 0.5) (layers *.Cu *.Mask))
-    (pad "" np_thru_hole circle (at 1.532737 0.865248 180) (size 0.6 0.6) (drill 0.5) (layers *.Cu *.Mask))
   )
   (footprint "Resistor_SMD:R_0603_1608Metric_Pad0.98x0.95mm_HandSolder" (layer "F.Cu")
@@
     )
     (pad "" np_thru_hole circle (at -1.532737 0.865248 270) (size 0.6 0.6) (drill 0.5) (layers *.Cu *.Mask))
+    (pad "" np_thru_hole circle (at 0 0.75 270) (size 0.6 0.6) (drill 0.5) (layers *.Cu *.Mask))
+    (pad "" np_thru_hole circle (at 1.532737 0.865248 270) (size 0.6 0.6) (drill 0.5) (layers *.Cu *.Mask))
     (pad "" np_thru_hole circle (at -0.768531 0.778853 270) (size 0.6 0.6) (drill 0.5) (layers *.Cu *.Mask))
     (pad "" np_thru_hole circle (at 0.768531 0.778853 270) (size 0.6 0.6) (drill 0.5) (layers *.Cu *.Mask))
-    (pad "" np_thru_hole circle (at 0 0.75 270) (size 0.6 0.6) (drill 0.5) (layers *.Cu *.Mask))
-    (pad "" np_thru_hole circle (at 1.532737 0.865248 270) (size 0.6 0.6) (drill 0.5) (layers *.Cu *.Mask))
   )
   (gr_line (start 13.55 2) (end 11.325 2) (layer "Edge.Cuts") (width 0.1))
@@
   (via (at -1.6 5.2) (size 0.8) (drill 0.4) (layers "F.Cu" "B.Cu") (net 5))
   (via (at 1.6 -5.4) (size 0.8) (drill 0.4) (layers "F.Cu" "B.Cu") (net 5))
-  (zone (net 1) (net_name "GND") (layer "F.Cu") (hatch edge 0.508)
+  (zone (net 5) (net_name "+3.3V") (layer "F.Cu") (hatch edge 0.508)
     (connect_pads (clearance 0.508))
     (min_thickness 0.254) (filled_areas_thickness no)
@@
     )
   )
-  (zone (net 5) (net_name "+3.3V") (layer "B.Cu") (hatch edge 0.508)
+  (zone (net 1) (net_name "GND") (layer "B.Cu") (hatch edge 0.508)
     (connect_pads (clearance 0.508))
     (min_thickness 0.254) (filled_areas_thickness no)

Commit message: BOM and fixed pcb
Routing:
- added copper zone on B.Cu, net +3.3V
- added copper zone on F.Cu, net GND
- removed copper zone on F.Cu, net +3.3V
- removed copper zone on B.Cu, net GND
Changed lines of the file:
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@@
   (via (at -1.6 5.2) (size 0.8) (drill 0.4) (layers "F.Cu" "B.Cu") (net 5))
   (via (at 1.6 -5.4) (size 0.8) (drill 0.4) (layers "F.Cu" "B.Cu") (net 5))
-  (zone (net 5) (net_name "+3.3V") (layer "F.Cu") (hatch edge 0.508)
+  (zone (net 1) (net_name "GND") (layer "F.Cu") (hatch edge 0.508)
     (connect_pads (clearance 0.508))
     (min_thickness 0.254) (filled_areas_thickness no)
@@
     )
   )
-  (zone (net 1) (net_name "GND") (layer "B.Cu") (hatch edge 0.508)
+  (zone (net 5) (net_name "+3.3V") (layer "B.Cu") (hatch edge 0.508)
     (connect_pads (clearance 0.508))
     (min_thickness 0.254) (filled_areas_thickness no)
